Commit message: Add files via upload

File: jazzy_ws/assets/dodo_daimao/urdf/dodo_daimao.urdf (robot description, URDF)
Before this commit: robot dodo_daimao, 11 links, 10 joints
Links:
- link body: geometry collision box size=0.27 0.21 0.1; visual mesh filename=../meshes/body.STL
- link foot_left: mass 0.0358036768207827 -> 0.035804; geometry collision box size=0.095 0.034 0.0655; visual mesh filename=../meshes/foot_left.STL
- link foot_right: geometry collision box size=0.095 0.034 0.0655; visual mesh filename=../meshes/foot_right.STL
- link foot_sole_left: geometry collision box size=0.095 0.022 0.005; visual mesh filename=../meshes/foot_sole_left.STL
- link foot_sole_right: geometry collision box size=0.095 0.022 0.005; visual mesh filename=../meshes/foot_sole_right.STL
- link hip_left: mass 0 -> 0.428645410212592; geometry collision box size=0.15 0.08 0.065; visual mesh filename=../meshes/hip_left.STL
- link hip_right: geometry collision box size=0.15 0.08 0.065; visual mesh filename=../meshes/hip_right.STL
- link lower_leg_left: mass 0.0729640311072434 -> 0.0729947991135356; geometry collision box size=0.046 0.037 0.23; visual mesh filename=../meshes/lower_leg_left.STL
- link lower_leg_right: geometry collision box size=0.046 0.037 0.23; visual mesh filename=../meshes/lower_leg_right.STL
- link upper_leg_left: mass 0.139831556786489 -> 0.13997; geometry collision box size=0.065 0.035 0.235; visual mesh filename=../meshes/upper_leg_left.STL
- link upper_leg_right: geometry collision box size=0.065 0.035 0.235; visual mesh filename=../meshes/upper_leg_right.STL
Joints:
- joint foot_sole_left: axis 0 0 0 -> (none); origin xyz=0.0136701751849855 0.00459982071533604 -0.0488007300265155 rpy=0 0 -3.14026372919282 -> xyz=0.0136701751849855 0.00459982071533604 -0.0488007300265155 rpy=0 0 0
- joint foot_sole_right: axis 0 0 0 -> (none)
